File: Harness TXX.kicad_sch (KiCad schematic)
At the start: 9 parts, among them J1 AnalogInp, J2 InpConn, J3 OutConn

Commit message: fixes
Connections:
- net +12V renamed +24V
- no-connect marks 38 -> 37
Other:
- sheet MCU: file 2023KicadLibrary\Standardized Subsheets\microcontroller.kicad_sch -> ..\..\2023KicadLibrary\Standardized Subsheets\microcontroller.kicad_sch
- sheet VRM: file 2023KicadLibrary\Standardized Subsheets\StandardizedVRMS.kicad_sch -> ..\..\2023KicadLibrary\Standardized Subsheets\vrmsv2.kicad_sch
- sheet VRM ports: added none; removed 12V_In_Unprotected, 12V_Out_Protected, 3V3_Out_Protected, 5V_Out_Protected

Commit message: made recommended adjustmetns
Parts:
- removed J1: AnalogInp, symbol Connector_Generic:Conn_01x08
- removed J2: InpConn, symbol Connector_Generic:Conn_01x08
- removed J3: OutConn, symbol Connector_Generic:Conn_01x08
- removed SWM_1: JS202011JCQN, SamacSys_Parts:JS202011JCQN, symbol LHRE Component Library:SW_DPDT
- added J1, J2, J3: Conn_01x06, symbol Connector_Generic:Conn_01x06
- added SW1, SW2: SW_SPDT, symbol Switch:SW_SPDT
Connections:
- net +24V: now also J1.4 (Pin_4), J2.4 (Pin_4), J3.4 (Pin_4)
- net +5V: now also J2.5 (Pin_5)
- net CAN+: now also J1.5 (Pin_5), J3.5 (Pin_5)
- net CAN-: now also J1.2 (Pin_2), J3.2 (Pin_2)
- net Extra1: now also J2.6 (Pin_6)
- net GND: now also J1.1 (Pin_1), J1.3 (Pin_3), J2.1 (Pin_1), J3.1 (Pin_1), J3.3 (Pin_3)
- net WheelIn1: now also J2.3 (Pin_3), SW1.1 (A), SW2.1 (A)
- net WheelIn2: now also J2.2 (Pin_2), SW1.3 (C), SW2.3 (C)
- new net PassThru1: J1.6 (Pin_6), SW1.2 (B)
- new net PassThru2: J3.6 (Pin_6), SW2.2 (B)
- no-connect marks 37 -> 40
Other:
- sheet MCU: file ..\..\2023KicadLibrary\Standardized Subsheets\microcontroller.kicad_sch -> 2023KicadLibrary\Standardized Subsheets\microcontroller.kicad_sch
- sheet VRM: file ..\..\2023KicadLibrary\Standardized Subsheets\vrmsv2.kicad_sch -> 2023KicadLibrary\Standardized Subsheets\vrmsv2.kicad_sch
