File: Harness TXX.kicad_sch (KiCad schematic)
At the start: 10 parts, among them J1 Conn_01x06, J2 Conn_01x06, J3 Conn_01x06, SW1 SW_SPDT, SW2 SW_SPDT

Commit message: Dakota's feedback
Parts:
- removed R1: Rterm, Resistor_SMD:R_0603_1608Metric_Pad0.98x0.95mm_HandSolder, symbol Device:R
- added R?: 120, Resistor_SMD:R_0603_1608Metric_Pad0.98x0.95mm_HandSolder, symbol Device:R
- added SW?: CAS-120B, symbol Switch:SW_SPDT
- J1, J2, J3: value Conn_01x06 -> DEUTSCH DT header
- SW1, SW2: value SW_SPDT -> CAS-120B
Connections:
- net CAN+: now also SW?.2 (B)
- net CAN-: now also R?.1
- new net: R?.2, SW?.1 (A)
- no-connect marks 40 -> 41

Commit message: Post Rylan Review Edits
Parts:
- removed D1, D2, D3, D4: SS36-E3_57T, DIOM7959X262N, symbol SamacSys_Parts:SS36-E3_57T
- removed J2: DEUTSCH DT header, symbol Connector_Generic:Conn_01x06
- removed R?: 120, Resistor_SMD:R_0603_1608Metric_Pad0.98x0.95mm_HandSolder, symbol Device:R
- removed SW?: CAS-120B, symbol Switch:SW_SPDT
- added D? (x4): SS36-E3_57T, DIOM7959X262N, symbol SamacSys_Parts:SS36-E3_57T
- added J3: DEUTSCH DT Data, symbol Connector_Generic:Conn_01x06
- J1: value DEUTSCH DT header -> DEUTSCH DT Inp
- J2: renamed from J3; value DEUTSCH DT header -> DEUTSCH DT Out
Connections:
- net +24V: now also J3.4 (Pin_4)
- net +3V3: now also D?.1, D?.1
- net +5V: now also J3.5 (Pin_5)
- net Extra1: now also J3.6 (Pin_6)
- net GND: now also D?.2, D?.2, J3.1 (Pin_1); no longer J1.3 (Pin_3), J2.3 (Pin_3)
- net WheelIn1: now also D?.1, D?.2, J3.3 (Pin_3)
- net WheelIn2: now also D?.1, D?.2, J3.2 (Pin_2)
- new net SHIELD: J1.3 (Pin_3), J2.3 (Pin_3)
- no-connect marks 41 -> 40
Other:
- note added: "Input Clamping Diodes"
- note added: "Input Connector"

Commit message: Workday progress
Parts:
- D1, D2, D3, D4: renamed from D?; value SS36-E3_57T -> SD0603S040S0R2; footprint DIOM7959X262N -> SamacSys_Parts:SD0603
- J1: footprint (none) -> Global Libraries:DT13-6P
- J2: renamed from J3; footprint (none) -> Global Libraries:DT13-6P
- J3: renamed from J2; footprint (none) -> Global Libraries:DT13-6P
- SW1, SW2: footprint (none) -> SamacSys_Parts:CAS120B
Connections:
- net PassThru1: now also J1.3 (Pin_3); no longer J1.6 (Pin_6)
- net PassThru2: now also J3.3 (Pin_3); no longer J3.6 (Pin_6)
- net SHIELD: now also J1.6 (Pin_6), J3.6 (Pin_6); no longer J1.3 (Pin_3), J3.3 (Pin_3)
- no-connect marks 40 -> 37
