File: Harness TXX.kicad_sch (KiCad schematic)
At the start: 9 parts, among them J1 DEUTSCH DT Inp, J2 DEUTSCH DT Data, J3 DEUTSCH DT Out, SW1 CAS-120B, SW2 CAS-120B

Commit message: Workday 12/4/22
Parts:
- added TP? (x4): TestPoint, symbol Connector:TestPoint
Connections:
- net GND: now also TP?.1, TP?.1, TP?.1, TP?.1
Changed lines of the file:
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@@
+    (pin "1")
+  )
+  (symbol (lib_id "power:GND") (at 16.51 57.15 0) (unit 1)
+    (in_bom yes) (on_board yes)
+    (property "Reference" "#PWR?" (id 0) (at 16.51 63.5 0)
+      (effects (font (size 1.27 1.27)) hide)
+    )
+    (property "Value" "GND" (id 1) (at 20.32 58.42 0))
+    (property "Footprint" "" (id 2) (at 16.51 57.15 0)
+      (effects (font (size 1.27 1.27)) hide)
+    )
+    (property "Datasheet" "" (id 3) (at 16.51 57.15 0)
+      (effects (font (size 1.27 1.27)) hide)
+    )
     (pin "1")
   )
@@
     (pin "1")
   )
+  (symbol (lib_id "Connector:TestPoint") (at 27.94 57.15 0) (unit 1)
+    (in_bom yes) (on_board yes) (fields_autoplaced)
+    (property "Reference" "TP?" (id 0) (at 29.337 52.9395 0)
+      (effects (font (size 1.27 1.27)) (justify left))
+    )
+    (property "Value" "TestPoint" (id 1) (at 29.337 55.7146 0)
+      (effects (font (size 1.27 1.27)) (justify left))
+    )
+    (property "Footprint" "" (id 2) (at 33.02 57.15 0)
+      (effects (font (size 1.27 1.27)) hide)
+    )
+    (property "Datasheet" "~" (id 3) (at 33.02 57.15 0)
+      (effects (font (size 1.27 1.27)) hide)
+    )
+    (pin "1")
+  )
   (symbol (lib_id "power:GND") (at 102.87 40.64 0) (mirror y) (unit 1)
     (in_bom yes) (on_board yes)
@@
     )
     (property "Datasheet" "" (id 3) (at 102.87 40.64 0)
+      (effects (font (size 1.27 1.27)) hide)
+    )
+    (pin "1")
+  )
+  (symbol (lib_id "Connector:TestPoint") (at 16.51 57.15 0) (unit 1)
+    (in_bom yes) (on_board yes) (fields_autoplaced)
+    (property "Reference" "TP?" (id 0) (at 17.907 52.9395 0)
+      (effects (font (size 1.27 1.27)) (justify left))
+    )
+    (property "Value" "TestPoint" (id 1) (at 17.907 55.7146 0)
+      (effects (font (size 1.27 1.27)) (justify left))
+    )
+    (property "Footprint" "" (id 2) (at 21.59 57.15 0)
+      (effects (font (size 1.27 1.27)) hide)
+    )
+    (property "Datasheet" "~" (id 3) (at 21.59 57.15 0)
       (effects (font (size 1.27 1.27)) hide)
     )
@@
     (pin "2")
   )
+  (symbol (lib_id "power:GND") (at 27.94 69.85 0) (unit 1)
+    (in_bom yes) (on_board yes)
+    (property "Reference" "#PWR?" (id 0) (at 27.94 76.2 0)
+      (effects (font (size 1.27 1.27)) hide)
+    )
+    (property "Value" "GND" (id 1) (at 31.75 71.12 0))
+    (property "Footprint" "" (id 2) (at 27.94 69.85 0)
+      (effects (font (size 1.27 1.27)) hide)
+    )
+    (property "Datasheet" "" (id 3) (at 27.94 69.85 0)
+      (effects (font (size 1.27 1.27)) hide)
+    )
+    (pin "1")
+  )
   (symbol (lib_id "Connector_Generic:Conn_01x06") (at 105.41 101.6 0) (mirror x) (unit 1)
     (in_bom yes) (on_board yes)
@@
     (pin "6")
   )
+  (symbol (lib_id "Connector:TestPoint") (at 16.51 69.85 0) (unit 1)
+    (in_bom yes) (on_board yes) (fields_autoplaced)
+    (property "Reference" "TP?" (id 0) (at 17.907 65.6395 0)
+      (effects (font (size 1.27 1.27)) (justify left))
+    )
+    (property "Value" "TestPoint" (id 1) (at 17.907 68.4146 0)
+      (effects (font (size 1.27 1.27)) (justify left))
+    )
+    (property "Footprint" "" (id 2) (at 21.59 69.85 0)
+      (effects (font (size 1.27 1.27)) hide)
+    )
+    (property "Datasheet" "~" (id 3) (at 21.59 69.85 0)
+      (effects (font (size 1.27 1.27)) hide)
+    )
+    (pin "1")
+  )
   (symbol (lib_id "Switch:SW_SPDT") (at 69.85 29.21 0) (unit 1)
     (in_bom yes) (on_board yes)
@@
     (pin "2")
   )
+  (symbol (lib_id "power:GND") (at 27.94 57.15 0) (unit 1)
+    (in_bom yes) (on_board yes)
+    (property "Reference" "#PWR?" (id 0) (at 27.94 63.5 0)
+      (effects (font (size 1.27 1.27)) hide)
+    )
+    (property "Value" "GND" (id 1) (at 31.75 58.42 0))
+    (property "Footprint" "" (id 2) (at 27.94 57.15 0)
+      (effects (font (size 1.27 1.27)) hide)
+    )
+    (property "Datasheet" "" (id 3) (at 27.94 57.15 0)
+      (effects (font (size 1.27 1.27)) hide)
+    )
+    (pin "1")
+  )
+  (symbol (lib_id "Connector:TestPoint") (at 27.94 69.85 0) (unit 1)
+    (in_bom yes) (on_board yes) (fields_autoplaced)
+    (property "Reference" "TP?" (id 0) (at 29.337 65.6395 0)
+      (effects (font (size 1.27 1.27)) (justify left))
+    )
+    (property "Value" "TestPoint" (id 1) (at 29.337 68.4146 0)
+      (effects (font (size 1.27 1.27)) (justify left))
+    )
+    (property "Footprint" "" (id 2) (at 33.02 69.85 0)
+      (effects (font (size 1.27 1.27)) hide)
+    )
+    (property "Datasheet" "~" (id 3) (at 33.02 69.85 0)
+      (effects (font (size 1.27 1.27)) hide)
+    )
+    (pin "1")
+  )
   (symbol (lib_id "power:GND") (at 105.41 149.86 0) (unit 1)
     (in_bom yes) (on_board yes)
@@
     (pin "1")
     (pin "2")
+  )
+  (symbol (lib_id "power:GND") (at 16.51 69.85 0) (unit 1)
+    (in_bom yes) (on_board yes)
+    (property "Reference" "#PWR?" (id 0) (at 16.51 76.2 0)
+      (effects (font (size 1.27 1.27)) hide)
+    )
+    (property "Value" "GND" (id 1) (at 20.32 71.12 0))
+    (property "Footprint" "" (id 2) (at 16.51 69.85 0)
+      (effects (font (size 1.27 1.27)) hide)
+    )
+    (property "Datasheet" "" (id 3) (at 16.51 69.85 0)
+      (effects (font (size 1.27 1.27)) hide)
+    )
+    (pin "1")
   )
   (sheet (at 40.64 57.15) (size 27.94 12.7)
@@
       (reference "#FLG04") (unit 1) (value "PWR_FLAG") (footprint "")
     )
-    (path "/3b53be70-8bbf-4fac-8f44-e59c6521e9a1/70562e2b-054a-4a0b-b5a5-933e5c1c68eb"
-      (reference "#FLG05") (unit 1) (value "PWR_FLAG") (footprint "")
-    )
     (path "/3b53be70-8bbf-4fac-8f44-e59c6521e9a1/2d4a2a6c-073d-45fb-a4ea-042f6d0945ef"
       (reference "#FLG06") (unit 1) (value "PWR_FLAG") (footprint "")
@@
       (reference "#PWR066") (unit 1) (value "GNDPWR") (footprint "")
     )
+    (path "/0c4507b5-720b-48a4-bec3-940f91c17d3d"
+      (reference "#PWR?") (unit 1) (value "GND") (footprint "")
+    )
+    (path "/5a9e383c-8df8-463f-b5fa-2bf773b28404"
+      (reference "#PWR?") (unit 1) (value "GND") (footprint "")
+    )
+    (path "/c93cd49c-b481-4da4-a2a8-b2ee484ca8d8"
+      (reference "#PWR?") (unit 1) (value "GND") (footprint "")
+    )
+    (path "/faae6525-a334-4e64-b32e-803caa067fb3"
+      (reference "#PWR?") (unit 1) (value "GND") (footprint "")
+    )
     (path "/2efde200-f5ff-4d23-9097-2b6180714d77/5eef7685-46e3-4490-b1c3-d367d5bf00e5/385351ea-5439-438d-bd65-1e74a98e8cb5"
       (reference "C1") (unit 1) (value "10uF") (footprint "Capacitor_SMD:C_0603_1608Metric_Pad1.08x0.95mm_HandSolder")
@@
       (reference "TP8") (unit 1) (value " ") (footprint "TestPoint:TestPoint_THTPad_1.0x1.0mm_Drill0.5mm")
     )
+    (path "/16770014-b0c5-4586-834e-2360f271364d"
+      (reference "TP?") (unit 1) (value "TestPoint") (footprint "")
+    )
+    (path "/1c0a24db-2b88-4f72-a8d4-d1ae65f4e55e"
+      (reference "TP?") (unit 1) (value "TestPoint") (footprint "")
+    )
+    (path "/6e11e5c3-3d6b-479d-844d-fab614dbf2de"
+      (reference "TP?") (unit 1) (value "TestPoint") (footprint "")
+    )
+    (path "/d08f9ed6-978b-4757-b454-b0bb3c3e1635"
+      (reference "TP?") (unit 1) (value "TestPoint") (footprint "")
+    )
     (path "/2efde200-f5ff-4d23-9097-2b6180714d77/5eef7685-46e3-4490-b1c3-d367d5bf00e5/8cd40687-f12d-4487-81ad-e4b3943431ac"

Commit message: Board wiring
Parts:
- removed SW2: CAS-120B, SamacSys_Parts:CAS120B, symbol Switch:SW_SPDT
- gave numbers to parts that had none: 4
Connections:
- net PassThru2 is gone; now on net PassThru: J3.3 (Pin_3)
- net PassThru1 renamed PassThru

Commit message: Had been modifying a file on my computer and not git on accident. Adding updated PCB to Git
Parts:
- J1, J2, J3: footprint Global Libraries:DT13-6P -> Connector_Molex:Molex_Micro-Fit_3.0_43045-0600_2x03_P3.00mm_Horizontal
- SW1: value CAS-120B -> SW_SPDT; footprint SamacSys_Parts:CAS120B -> SamacSys_Parts:CAS120A1
- TP1, TP2, TP3, TP4: footprint (none) -> TestPoint:TestPoint_Plated_Hole_D3.0mm
